File: doc/schematics/licht.brd (EAGLE design)
At the start: 65.3 x 36.2 mm, 25 parts, among them Q1 MOSFET-NCHANNELFQP30N06L, Q2 MOSFET-PCHANNELSMD

Commit message: toller state
Parts:
- D1: value (none) -> SMD ZD 16; device diode:SOT223 -> diode:SOT23
- Q2: value MOSFET-PCHANNELSMD -> IRFML8244
- moved F1 71.5 mm to (49.5, 5.33), flipped to the bottom, turned to 90 degrees
- moved R3 66.4 mm to (50.8, 12.4), turned to 180 degrees
- moved D1 58.2 mm to (45.2, 13.2), turned to 90 degrees
- moved Q2 50.7 mm to (44.5, 9.14), turned to 180 degrees
Connections:
- net V+: now also D1.3; no longer D1.4
Routing:
- net V+: track 18.1 -> 27.1 mm
- net N$5: track 0.00 -> 6.75 mm
- net N$3: track 2.48 -> 7.36 mm
- net N$4: track 0.00 -> 2.71 mm
Changed lines of the file:
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@@
 <attribute name="OC_FARNELL" value="unknown" x="6.604" y="17.78" size="1.778" layer="28" rot="MR270" display="off"/>
 </element>
-<element name="Q2" library="SparkFun-DiscreteSemi" package="SOT23-3" value="MOSFET-PCHANNELSMD" x="-5.334" y="-0.508"/>
-<element name="D1" library="diode" package="SOT223" value="" x="-11.938" y="2.286"/>
-<element name="R3" library="rcl" package="R0805" value="100k" x="-13.208" y="-5.08"/>
+<element name="Q2" library="SparkFun-DiscreteSemi" package="SOT23-3" value="IRFML8244" x="44.45" y="9.144" rot="R180">
+<attribute name="PROD_ID" value="TRANS-08285" x="44.45" y="9.144" size="1.778" layer="27" rot="R180" display="off"/>
+</element>
+<element name="D1" library="diode" package="SOT23" value="SMD ZD 16" x="45.212" y="13.208" rot="R90"/>
+<element name="R3" library="rcl" package="R0805" value="100k" x="50.8" y="12.446" rot="R180"/>
 <element name="ROTARY" library="con-lstb" package="MA04-1" value="" x="22.098" y="27.686" rot="MR0">
 <attribute name="OC_NEWARK" value="unknown" x="22.098" y="27.686" size="1.778" layer="28" rot="MR0" display="off"/>
@@
 <element name="R2" library="rcl" package="R0805" value="10k" x="20.828" y="32.004" rot="R270"/>
 <element name="R4" library="rcl" package="R0805" value="10k" x="23.368" y="32.004" rot="R270"/>
-<element name="F1" library="sprawl" package="PTF45" value="" x="-21.844" y="1.524">
-<attribute name="OC_NEWARK" value="unknown" x="-21.844" y="1.524" size="1.778" layer="27" display="off"/>
-<attribute name="MPN" value="" x="-21.844" y="1.524" size="1.778" layer="27" display="off"/>
-<attribute name="MF" value="" x="-21.844" y="1.524" size="1.778" layer="27" display="off"/>
-<attribute name="OC_FARNELL" value="unknown" x="-21.844" y="1.524" size="1.778" layer="27" display="off"/>
-<attribute name="OC_REICHELT" value="PL 122100" x="-21.844" y="1.524" size="1.778" layer="27" display="off"/>
+<element name="F1" library="sprawl" package="PTF45" value="" x="49.53" y="5.334" rot="MR90">
+<attribute name="OC_NEWARK" value="unknown" x="49.53" y="5.334" size="1.778" layer="28" rot="MR90" display="off"/>
+<attribute name="MPN" value="" x="49.53" y="5.334" size="1.778" layer="28" rot="MR90" display="off"/>
+<attribute name="MF" value="" x="49.53" y="5.334" size="1.778" layer="28" rot="MR90" display="off"/>
+<attribute name="OC_FARNELL" value="unknown" x="49.53" y="5.334" size="1.778" layer="28" rot="MR90" display="off"/>
+<attribute name="OC_REICHELT" value="PL 122100" x="49.53" y="5.334" size="1.778" layer="28" rot="MR90" display="off"/>
 </element>
 </elements>
@@
 <contactref element="ROTARY" pad="1"/>
 <contactref element="ISP" pad="1"/>
-<wire x1="5.842" y1="6.538" x2="-14.158" y2="-5.08" width="0" layer="19" extent="1-1"/>
 </signal>
 <signal name="+3V3">
@@
 <signal name="N$3">
 <contactref element="X_PWR" pad="2"/>
-<wire x1="59.4821" y1="5.334" x2="61.239" y2="3.5771" width="1.778" layer="1"/>
 <contactref element="F1" pad="1"/>
-<wire x1="-21.844" y1="6.604" x2="59.4821" y2="5.334" width="0" layer="19" extent="1-1"/>
+<wire x1="61.239" y1="3.5771" x2="59.4821" y2="5.334" width="1.778" layer="1"/>
+<wire x1="59.4821" y1="5.334" x2="54.61" y2="5.334" width="1.778" layer="1"/>
 </signal>
 <signal name="N$4">
 <contactref element="Q2" pad="3"/>
 <contactref element="F1" pad="2"/>
-<wire x1="-5.334" y1="0.592" x2="-21.844" y2="-3.556" width="0" layer="19" extent="1-1"/>
+<wire x1="44.45" y1="8.044" x2="44.45" y2="5.334" width="1.778" layer="1"/>
 </signal>
 <signal name="V+">
@@
 <contactref element="C6" pad="1"/>
 <contactref element="Q2" pad="2"/>
-<contactref element="D1" pad="4"/>
+<contactref element="D1" pad="3"/>
 <contactref element="L1" pad="1"/>
 <wire x1="30.54" y1="14.351" x2="39.407" y2="14.351" width="0.4064" layer="1"/>
 <wire x1="39.407" y1="14.351" x2="39.624" y2="14.568" width="0.4064" layer="1"/>
+<wire x1="44.112" y1="13.208" x2="43.434" y2="13.208" width="1.778" layer="1"/>
+<wire x1="43.434" y1="13.208" x2="39.624" y2="13.208" width="1.778" layer="1"/>
+<wire x1="39.624" y1="13.208" x2="39.624" y2="14.568" width="1.778" layer="1"/>
+<wire x1="43.5" y1="10.144" x2="43.434" y2="10.144" width="1.778" layer="1"/>
+<wire x1="43.434" y1="10.144" x2="43.434" y2="13.208" width="1.778" layer="1"/>
 <wire x1="31.176" y1="10.922" x2="30.54" y2="14.351" width="0" layer="19" extent="1-1"/>
 <wire x1="23.114" y1="5.334" x2="31.176" y2="10.922" width="0" layer="19" extent="1-1"/>
-<wire x1="-4.384" y1="-1.508" x2="14.7828" y2="6.8834" width="0" layer="19" extent="1-1"/>
-<wire x1="-11.938" y1="5.385" x2="-4.384" y2="-1.508" width="0" layer="19" extent="1-1"/>
 </signal>
 <signal name="N$5">
@@
 <contactref element="D1" pad="1"/>
 <contactref element="R3" pad="2"/>
-<wire x1="-14.249" y1="-0.813" x2="-12.258" y2="-5.08" width="0" layer="19" extent="1-1"/>
-<wire x1="-6.284" y1="-1.508" x2="-12.258" y2="-5.08" width="0" layer="19" extent="1-1"/>
+<wire x1="45.4" y1="10.144" x2="46.312" y2="10.144" width="0.4064" layer="1"/>
+<wire x1="46.312" y1="10.144" x2="46.312" y2="12.258" width="0.4064" layer="1"/>
+<wire x1="46.312" y1="12.258" x2="49.85" y2="12.258" width="0.4064" layer="1"/>
+<wire x1="49.85" y1="12.258" x2="49.85" y2="12.446" width="0.4064" layer="1"/>
 </signal>
 <signal name="ROTBTN">

Commit message: toller state
Parts:
- moved IC1 14.5 mm to (26.2, 4.83)
- moved C2 14.5 mm to (32.8, 4.83)
- moved C4 14.5 mm to (37.6, 4.32)
- moved C1 13.7 mm to (19.6, 4.83), turned to 180 degrees
- moved Q1 6.60 mm to (58.7, 18.8)
- moved C6 4.89 mm to (34.5, 13.2), turned to 270 degrees
Routing:
- net FET1: track 0.00 -> 26.9 mm
- net N$2: track 0.00 -> 9.47 mm
- net V+: track 27.1 -> 36.1 mm
- net +3V3: track 76.1 -> 67.2 mm
- net GND: track 34.0 -> 30.8 mm, vias 2 -> 4
Changed lines of the file:
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@@
 <elements>
 <element name="U$1" library="LPC800" package="SOIC20WIDE" value="LPC812M101JD20" x="16.764" y="18.796" rot="R90"/>
-<element name="IC1" library="SparkFun-PowerIC" package="SOT223" value="" x="11.684" y="4.572" rot="R90"/>
+<element name="IC1" library="SparkFun-PowerIC" package="SOT223" value="" x="26.162" y="4.826" rot="R90"/>
 <element name="C3" library="rcl" package="C0805" value="100n" x="17.526" y="10.668" rot="R180"/>
 <element name="X_PWR" library="con-phoenix-508" package="MKDSN1,5/2-5,08" value="MKDSN1,5/2-5,08" x="61.214" y="6.096" rot="R270">
@@
 <attribute name="OC_FARNELL" value="1792903" x="43.434" y="-14.224" size="1.778" layer="27" rot="R270" display="off"/>
 </element>
-<element name="Q1" library="SparkFun-DiscreteSemi" package="TO220V" value="MOSFET-NCHANNELFQP30N06L" x="52.07" y="18.796" rot="MR180">
-<attribute name="PROD_ID" value="TRANS-10060" x="68.58" y="58.166" size="1.778" layer="28" rot="MR180" display="off"/>
+<element name="Q1" library="SparkFun-DiscreteSemi" package="TO220V" value="MOSFET-NCHANNELFQP30N06L" x="58.674" y="18.796" rot="MR180">
+<attribute name="PROD_ID" value="TRANS-10060" x="75.184" y="58.166" size="1.778" layer="28" rot="MR180" display="off"/>
 </element>
 <element name="X_LED" library="con-phoenix-508" package="MKDSN1,5/2-5,08" value="MKDSN1,5/2-5,08" x="61.214" y="29.718" rot="R270">
@@
 <attribute name="OC_FARNELL" value="1792903" x="32.004" y="9.398" size="1.778" layer="27" rot="R270" display="off"/>
 </element>
-<element name="C1" library="rcl" package="C0805" value="4u7" x="5.842" y="5.588" rot="R90"/>
-<element name="C2" library="rcl" package="C0805" value="100n" x="18.288" y="4.572" rot="R270"/>
-<element name="C4" library="rcl" package="E2,5-6" value="10u" x="23.114" y="4.064" rot="MR270"/>
+<element name="C1" library="rcl" package="C0805" value="4u7" x="19.558" y="4.826" rot="R180"/>
+<element name="C2" library="rcl" package="C0805" value="100n" x="32.766" y="4.826" rot="R270"/>
+<element name="C4" library="rcl" package="E2,5-6" value="10u" x="37.592" y="4.318" rot="MR270"/>
 <element name="U$2" library="florolf" package="SOIC8" value="IR4427SOIC8" x="27.94" y="14.986" rot="R270"/>
-<element name="C6" library="rcl" package="C0805" value="100n" x="30.226" y="10.922" rot="R180"/>
+<element name="C6" library="rcl" package="C0805" value="100n" x="34.544" y="13.208" rot="R270"/>
 <element name="L1" library="florolf" package="PISR-BIGPAD" value="1u" x="39.624" y="23.368" rot="R90"/>
 <element name="C7" library="florolf" package="PANASONIC_D-BIGPAD" value="100u" x="51.054" y="28.702" rot="R90"/>
@@
 <contactref element="NRF" pad="1"/>
 <contactref element="X_PWR" pad="1"/>
-<via x="30.734" y="32.258" extent="1-16" drill="0.6"/>
-<via x="60.198" y="15.24" extent="1-16" drill="0.6"/>
-<wire x1="30.734" y1="32.258" x2="60.198" y2="15.24" width="0.4064" layer="16"/>
+<via x="34.798" y="9.144" extent="1-16" drill="0.6"/>
+<via x="60.706" y="13.462" extent="1-16" drill="0.6"/>
+<wire x1="34.798" y1="9.144" x2="60.706" y2="13.462" width="0.4064" layer="16"/>
 <contactref element="R3" pad="1"/>
 <contactref element="ROTARY" pad="1"/>
 <contactref element="ISP" pad="1"/>
+<via x="50.546" y="20.828" extent="1-16" drill="0.6"/>
+<via x="50.546" y="16.256" extent="1-16" drill="0.6"/>
+<wire x1="50.546" y1="20.828" x2="50.546" y2="16.256" width="0.4064" layer="16"/>
 </signal>
 <signal name="+3V3">
@@
 <contactref element="U$1" pad="15"/>
 <contactref element="C3" pad="1"/>
-<wire x1="14.7828" y1="4.572" x2="8.585" y2="4.572" width="0.4064" layer="1"/>
+<wire x1="29.2608" y1="4.826" x2="23.063" y2="4.826" width="0.4064" layer="1"/>
 <contactref element="C5" pad="1"/>
 <contactref element="IR1" pad="VS"/>
@@
 <wire x1="7.62" y1="29.464" x2="7.62" y2="26.736" width="0.4064" layer="1"/>
 <wire x1="7.62" y1="26.736" x2="7.554" y2="26.67" width="0.4064" layer="1"/>
-<wire x1="18.476" y1="10.668" x2="18.476" y2="8.382" width="0.4064" layer="1"/>
-<wire x1="18.476" y1="8.382" x2="9.652" y2="8.382" width="0.4064" layer="1"/>
-<wire x1="9.652" y1="8.382" x2="8.636" y2="7.366" width="0.4064" layer="1"/>
-<wire x1="8.636" y1="7.366" x2="8.636" y2="4.623" width="0.4064" layer="1"/>
-<wire x1="8.636" y1="4.623" x2="8.585" y2="4.572" width="0.4064" layer="1"/>
-<wire x1="5.842" y1="4.638" x2="8.519" y2="4.638" width="0.4064" layer="1"/>
-<wire x1="8.519" y1="4.638" x2="8.585" y2="4.572" width="0.4064" layer="1"/>
 <wire x1="11.7348" y1="19.431" x2="14.732" y2="19.431" width="0.4064" layer="1"/>
 <wire x1="14.732" y1="19.431" x2="18.476" y2="19.431" width="0.4064" layer="1"/>
@@
 <wire x1="14.732" y1="31.176" x2="14.732" y2="19.431" width="0.4064" layer="1"/>
 <wire x1="14.798" y1="31.242" x2="16.51" y2="32.954" width="0.4064" layer="1"/>
+<wire x1="20.508" y1="4.826" x2="23.063" y2="4.826" width="0.4064" layer="1"/>
+<wire x1="20.508" y1="4.826" x2="20.508" y2="8.636" width="0.4064" layer="1"/>
+<wire x1="20.508" y1="8.636" x2="18.476" y2="10.668" width="0.4064" layer="1"/>
 </signal>
 <signal name="FET1">
 <contactref element="Q1" pad="1"/>
 <contactref element="U$2" pad="7"/>
-<wire x1="30.54" y1="15.621" x2="49.53" y2="18.796" width="0" layer="19" extent="1-1"/>
+<wire x1="30.54" y1="15.621" x2="32.385" y2="15.621" width="0.4064" layer="1"/>
+<wire x1="32.385" y1="15.621" x2="35.56" y2="18.796" width="0.4064" layer="1"/>
+<wire x1="35.56" y1="18.796" x2="56.134" y2="18.796" width="0.4064" layer="1"/>
 </signal>
 <signal name="SWCLK">
@@
 <contactref element="Q1" pad="2"/>
 <contactref element="X_LED" pad="2"/>
-<wire x1="52.07" y1="18.796" x2="61.239" y2="27.1991" width="0" layer="19" extent="1-1"/>
+<wire x1="58.674" y1="18.796" x2="58.674" y2="24.6341" width="1.778" layer="1"/>
+<wire x1="58.674" y1="24.6341" x2="61.239" y2="27.1991" width="1.778" layer="1"/>
 </signal>
 <signal name="N$3">
@@
 <contactref element="C2" pad="1"/>
 <contactref element="C4" pad="+"/>
-<wire x1="18.288" y1="5.522" x2="18.476" y2="5.334" width="0.4064" layer="1"/>
-<wire x1="14.7828" y1="6.8834" x2="16.9266" y2="6.8834" width="0.4064" layer="1"/>
-<wire x1="16.9266" y1="6.8834" x2="18.288" y2="5.522" width="0.4064" layer="1"/>
-<wire x1="18.476" y1="5.334" x2="23.114" y2="5.334" width="0.4064" layer="1"/>
 <contactref element="U$2" pad="6"/>
 <contactref element="C6" pad="1"/>
@@
 <contactref element="D1" pad="3"/>
 <contactref element="L1" pad="1"/>
-<wire x1="30.54" y1="14.351" x2="39.407" y2="14.351" width="0.4064" layer="1"/>
 <wire x1="39.407" y1="14.351" x2="39.624" y2="14.568" width="0.4064" layer="1"/>
 <wire x1="44.112" y1="13.208" x2="43.434" y2="13.208" width="1.778" layer="1"/>
@@
 <wire x1="43.5" y1="10.144" x2="43.434" y2="10.144" width="1.778" layer="1"/>
 <wire x1="43.434" y1="10.144" x2="43.434" y2="13.208" width="1.778" layer="1"/>
-<wire x1="31.176" y1="10.922" x2="30.54" y2="14.351" width="0" layer="19" extent="1-1"/>
-<wire x1="23.114" y1="5.334" x2="31.176" y2="10.922" width="0" layer="19" extent="1-1"/>
+<wire x1="37.592" y1="5.588" x2="39.624" y2="7.62" width="0.4064" layer="1"/>
+<wire x1="39.624" y1="7.62" x2="39.624" y2="13.208" width="0.4064" layer="1"/>
+<wire x1="32.766" y1="5.776" x2="32.954" y2="5.588" width="0.4064" layer="1"/>
+<wire x1="32.954" y1="5.588" x2="37.592" y2="5.588" width="0.4064" layer="1"/>
+<wire x1="32.766" y1="5.776" x2="31.4046" y2="7.1374" width="0.4064" layer="1"/>
+<wire x1="31.4046" y1="7.1374" x2="29.2608" y2="7.1374" width="0.4064" layer="1"/>
+<wire x1="34.544" y1="14.158" x2="34.351" y2="14.351" width="0.4064" layer="1"/>
+<wire x1="34.351" y1="14.351" x2="30.54" y2="14.351" width="0.4064" layer="1"/>
+<wire x1="34.544" y1="14.158" x2="39.214" y2="14.158" width="0.4064" layer="1"/>
+<wire x1="39.214" y1="14.158" x2="39.624" y2="14.568" width="0.4064" layer="1" curve="90"/>
 </signal>
 <signal name="N$5">

Commit message: fast fertig
Routing:
- net SCK: track 14.1 -> 19.5 mm
- net CE: track 28.4 -> 33.4 mm
- net +3V3: track 67.2 -> 70.2 mm
- net SWDIO: track 9.56 -> 11.9 mm
- net MISO: track 8.69 -> 10.8 mm
- net V+: track 36.1 -> 38.0 mm
- net FET1: track 26.9 -> 28.8 mm
- net SWCLK: track 9.03 -> 10.6 mm
- net IROUT: track 5.39 -> 5.92 mm
