File: doc/schematics/licht.brd (EAGLE design)
At the start: 65.3 x 36.2 mm, 25 parts, among them Q1 MOSFET-NCHANNELFQP30N06L, Q2 IRFML8244

Commit message: Lauter neue Teile
Parts:
- removed D1: SMD ZD 16, diode:SOT23
- removed IC1: (no value), SparkFun-PowerIC:SOT223
- removed R3: 100k, rcl:R0805
- added IC2: (no value), sprawl:TO252
- C7: device florolf:PANASONIC_D-BIGPAD -> florolf:E2,5-5
- Q2: value IRFML8244 -> IRF7416; device SparkFun-DiscreteSemi:SOT23-3 -> sprawl:SO8
- moved C1 8.46 mm to (25.9, 10.4), turned to 0 degrees
- moved Q2 3.64 mm to (47.8, 10.7), turned to 270 degrees
- moved C7 2.34 mm to (50.5, 31.0), flipped to the bottom, turned to 270 degrees
Connections:
- removed net N$5: D1.1, Q2.1, R3.2
- net +3V3: now also IC2.3; no longer IC1.2, IC1.4
- net GND: now also IC2.2, Q2.4; no longer IC1.1, R3.1
- net N$4: now also Q2.5, Q2.6, Q2.7, Q2.8; no longer Q2.3
- net V+: now also IC2.1, Q2.1, Q2.3; no longer D1.3, IC1.3
Routing:
- net N$4: track 2.71 -> 13.1 mm
- net +3V3: track 70.2 -> 63.3 mm
- net N$5: track 6.75 -> 0.00 mm
- net V+: track 38.0 -> 41.8 mm
- added copper zone on layer 1, net V+
Changed lines of the file:
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@@
 <wire x1="65.258" y1="36.246" x2="0" y2="36.246" width="0" layer="20"/>
 <wire x1="0" y1="36.246" x2="0" y2="0" width="0" layer="20"/>
-<hole x="4.826" y="4.826" drill="0.6"/>
-<hole x="30.988" y="32.258" drill="0.6"/>
 </plain>
 <attributes>
@@
 <elements>
 <element name="U$1" library="LPC800" package="SOIC20WIDE" value="LPC812M101JD20" x="16.764" y="18.796" rot="R90"/>
-<element name="IC1" library="SparkFun-PowerIC" package="SOT223" value="" x="26.162" y="4.826" rot="R90"/>
 <element name="C3" library="rcl" package="C0805" value="100n" x="17.526" y="10.668" rot="R180"/>
 <element name="X_PWR" library="con-phoenix-508" package="MKDSN1,5/2-5,08" value="MKDSN1,5/2-5,08" x="61.214" y="6.096" rot="R270">
@@
 <attribute name="OC_FARNELL" value="1792903" x="32.004" y="9.398" size="1.778" layer="27" rot="R270" display="off"/>
 </element>
-<element name="C1" library="rcl" package="C0805" value="4u7" x="19.558" y="4.826" rot="R180"/>
+<element name="C1" library="rcl" package="C0805" value="4u7" x="25.908" y="10.414"/>
 <element name="C2" library="rcl" package="C0805" value="100n" x="32.766" y="4.826" rot="R270"/>
 <element name="C4" library="rcl" package="E2,5-6" value="10u" x="37.592" y="4.318" rot="MR270"/>
@@
 <element name="C6" library="rcl" package="C0805" value="100n" x="34.544" y="13.208" rot="R270"/>
 <element name="L1" library="florolf" package="PISR-BIGPAD" value="1u" x="39.624" y="23.368" rot="R90"/>
-<element name="C7" library="florolf" package="PANASONIC_D-BIGPAD" value="100u" x="51.054" y="28.702" rot="R90"/>
+<element name="C7" library="florolf" package="E2,5-5" value="100u" x="50.546" y="30.988" rot="MR270"/>
 <element name="IR1" library="tsop1736" package="TSOP17_TB1" value="TSOP1736TB1" x="8.89" y="29.464" rot="MR90">
 <attribute name="OC_NEWARK" value="unknown" x="8.89" y="29.464" size="1.778" layer="28" rot="MR90" display="off"/>
@@
 <attribute name="OC_FARNELL" value="unknown" x="6.604" y="17.78" size="1.778" layer="28" rot="MR270" display="off"/>
 </element>
-<element name="Q2" library="SparkFun-DiscreteSemi" package="SOT23-3" value="IRFML8244" x="44.45" y="9.144" rot="R180">
-<attribute name="PROD_ID" value="TRANS-08285" x="44.45" y="9.144" size="1.778" layer="27" rot="R180" display="off"/>
-</element>
-<element name="D1" library="diode" package="SOT23" value="SMD ZD 16" x="45.212" y="13.208" rot="R90"/>
-<element name="R3" library="rcl" package="R0805" value="100k" x="50.8" y="12.446" rot="R180"/>
 <element name="ROTARY" library="con-lstb" package="MA04-1" value="" x="22.098" y="27.686" rot="MR0">
 <attribute name="OC_NEWARK" value="unknown" x="22.098" y="27.686" size="1.778" layer="28" rot="MR0" display="off"/>
@@
 <attribute name="OC_REICHELT" value="PL 122100" x="49.53" y="5.334" size="1.778" layer="28" rot="MR90" display="off"/>
 </element>
+<element name="IC2" library="sprawl" package="TO252" value="" x="20.32" y="5.334" rot="R90">
+<attribute name="OC_REICHELT" value="TS 2940 CP33" x="20.32" y="5.334" size="1.778" layer="27" rot="R90" display="off"/>
+</element>
+<element name="Q2" library="sprawl" package="SO8" value="IRF7416" x="47.752" y="10.668" rot="R270"/>
 </elements>
 <signals>
 <signal name="GND">
-<contactref element="IC1" pad="1"/>
 <contactref element="C1" pad="2"/>
 <contactref element="C2" pad="2"/>
@@
 <via x="60.706" y="13.462" extent="1-16" drill="0.6"/>
 <wire x1="34.798" y1="9.144" x2="60.706" y2="13.462" width="0.4064" layer="16"/>
-<contactref element="R3" pad="1"/>
 <contactref element="ROTARY" pad="1"/>
 <contactref element="ISP" pad="1"/>
@@
 <via x="50.546" y="16.256" extent="1-16" drill="0.6"/>
 <wire x1="50.546" y1="20.828" x2="50.546" y2="16.256" width="0.4064" layer="16"/>
-<polygon width="0.4064" layer="1">
+<polygon width="0.4064" layer="1" rank="2">
 <vertex x="-4.826" y="43.434"/>
 <vertex x="70.104" y="43.434"/>
@@
 <vertex x="-4.826" y="-6.604"/>
 </polygon>
+<contactref element="IC2" pad="2"/>
+<contactref element="Q2" pad="4"/>
 </signal>
 <signal name="+3V3">
-<contactref element="IC1" pad="2"/>
-<contactref element="IC1" pad="4"/>
 <contactref element="C1" pad="1"/>
 <contactref element="U$1" pad="15"/>
 <contactref element="C3" pad="1"/>
-<wire x1="29.2608" y1="4.826" x2="23.063" y2="4.826" width="0.4064" layer="1"/>
 <contactref element="C5" pad="1"/>
 <contactref element="IR1" pad="VS"/>
@@
 <wire x1="20.828" y1="32.954" x2="23.368" y2="32.954" width="0.4064" layer="1"/>
 <wire x1="14.732" y1="30.988" x2="14.732" y2="19.431" width="0.4064" layer="1"/>
-<wire x1="20.508" y1="4.826" x2="23.063" y2="4.826" width="0.4064" layer="1"/>
-<wire x1="20.508" y1="4.826" x2="20.508" y2="10.668" width="0.4064" layer="1"/>
-<wire x1="20.508" y1="10.668" x2="18.476" y2="10.668" width="0.4064" layer="1"/>
 <wire x1="7.62" y1="29.464" x2="7.62" y2="30.988" width="0.4064" layer="1"/>
 <wire x1="7.62" y1="30.988" x2="14.732" y2="30.988" width="0.4064" layer="1"/>
 <wire x1="18.288" y1="32.954" x2="14.732" y2="32.954" width="0.4064" layer="1"/>
 <wire x1="14.732" y1="32.954" x2="14.732" y2="30.988" width="0.4064" layer="1"/>
+<contactref element="IC2" pad="3"/>
+<wire x1="25.12" y1="7.614" x2="25.12" y2="10.414" width="0.4064" layer="1"/>
+<wire x1="25.12" y1="10.414" x2="24.958" y2="10.414" width="0.4064" layer="1"/>
+<wire x1="24.958" y1="10.414" x2="18.476" y2="10.414" width="0.4064" layer="1"/>
+<wire x1="18.476" y1="10.414" x2="18.476" y2="10.668" width="0.4064" layer="1"/>
 </signal>
 <signal name="FET1">
@@
 <contactref element="L1" pad="2"/>
 <contactref element="C7" pad="+"/>
-<wire x1="39.624" y1="32.168" x2="50.988" y2="32.168" width="1.778" layer="1"/>
-<wire x1="50.988" y1="32.168" x2="51.054" y2="32.102" width="1.016" layer="1"/>
-<wire x1="51.054" y1="32.102" x2="61.0619" y2="32.102" width="1.778" layer="1"/>
-<wire x1="61.0619" y1="32.102" x2="61.239" y2="32.2791" width="1.778" layer="1"/>
+<wire x1="39.624" y1="32.168" x2="50.546" y2="32.168" width="1.778" layer="1"/>
+<wire x1="50.546" y1="32.168" x2="50.546" y2="32.258" width="1.778" layer="1"/>
+<wire x1="50.546" y1="32.258" x2="61.239" y2="32.258" width="1.778" layer="1"/>
+<wire x1="61.239" y1="32.258" x2="61.239" y2="32.2791" width="1.778" layer="1"/>
 </signal>
 <signal name="ROT2">
@@
 </signal>
 <signal name="N$4">
-<contactref element="Q2" pad="3"/>
 <contactref element="F1" pad="2"/>
-<wire x1="44.45" y1="8.044" x2="44.45" y2="5.334" width="1.778" layer="1"/>
+<contactref element="Q2" pad="5"/>
+<contactref element="Q2" pad="8"/>
+<contactref element="Q2" pad="7"/>
+<contactref element="Q2" pad="6"/>
+<wire x1="44.45" y1="5.334" x2="50.352" y2="5.334" width="1.778" layer="1"/>
+<wire x1="50.352" y1="5.334" x2="50.352" y2="8.763" width="1.778" layer="1"/>
+<wire x1="50.352" y1="8.763" x2="50.352" y2="10.033" width="1.778" layer="1"/>
+<wire x1="50.352" y1="10.033" x2="50.352" y2="11.303" width="1.778" layer="1"/>
+<wire x1="50.352" y1="11.303" x2="50.352" y2="12.573" width="1.778" layer="1"/>
 </signal>
 <signal name="V+">
-<contactref element="IC1" pad="3"/>
 <contactref element="C2" pad="1"/>
 <contactref element="C4" pad="+"/>
 <contactref element="U$2" pad="6"/>
 <contactref element="C6" pad="1"/>
-<contactref element="Q2" pad="2"/>
-<contactref element="D1" pad="3"/>
 <contactref element="L1" pad="1"/>
 <wire x1="39.407" y1="14.351" x2="39.624" y2="14.568" width="0.4064" layer="1"/>
-<wire x1="44.112" y1="13.208" x2="43.434" y2="13.208" width="1.778" layer="1"/>
-<wire x1="43.434" y1="13.208" x2="39.624" y2="13.208" width="1.778" layer="1"/>
 <wire x1="39.624" y1="13.208" x2="39.624" y2="14.568" width="1.778" layer="1"/>
-<wire x1="43.5" y1="10.144" x2="43.434" y2="10.144" width="1.778" layer="1"/>
-<wire x1="43.434" y1="10.144" x2="43.434" y2="13.208" width="1.778" layer="1"/>
 <wire x1="32.766" y1="5.776" x2="32.954" y2="5.588" width="0.4064" layer="1"/>
 <wire x1="32.954" y1="5.588" x2="37.592" y2="5.588" width="0.4064" layer="1"/>
@@
 <wire x1="39.214" y1="14.158" x2="39.624" y2="14.568" width="0.4064" layer="1" curve="90"/>
 <wire x1="37.592" y1="5.588" x2="39.624" y2="5.588" width="0.4064" layer="1"/>
-<wire x1="39.624" y1="5.588" x2="39.624" y2="13.208" width="0.4064" layer="1"/>
-<wire x1="32.766" y1="5.776" x2="32.766" y2="7.1374" width="0.4064" layer="1"/>
-<wire x1="32.766" y1="7.1374" x2="29.2608" y2="7.1374" width="0.4064" layer="1"/>
-</signal>
-<signal name="N$5">
+<wire x1="39.624" y1="5.588" x2="39.624" y2="12.954" width="0.4064" layer="1"/>
+<contactref element="IC2" pad="1"/>
+<wire x1="39.624" y1="12.954" x2="39.624" y2="13.208" width="0.4064" layer="1"/>
+<wire x1="32.766" y1="5.776" x2="28.702" y2="5.776" width="0.4064" layer="1"/>
+<wire x1="28.702" y1="5.776" x2="28.702" y2="3.054" width="0.4064" layer="1"/>
+<wire x1="28.702" y1="3.054" x2="25.12" y2="3.054" width="0.4064" layer="1"/>
 <contactref element="Q2" pad="1"/>
-<contactref element="D1" pad="1"/>
-<contactref element="R3" pad="2"/>
-<wire x1="45.4" y1="10.144" x2="46.312" y2="10.144" width="0.4064" layer="1"/>
-<wire x1="46.312" y1="10.144" x2="46.312" y2="12.258" width="0.4064" layer="1"/>
-<wire x1="46.312" y1="12.258" x2="49.85" y2="12.258" width="0.4064" layer="1"/>
-<wire x1="49.85" y1="12.258" x2="49.85" y2="12.446" width="0.4064" layer="1"/>
+<contactref element="Q2" pad="2"/>
+<contactref element="Q2" pad="3"/>
+<polygon width="0.254" layer="1" thermals="no">
+<vertex x="39.878" y="14.224"/>
+<vertex x="47.244" y="14.224"/>
+<vertex x="47.244" y="9.652"/>
+<vertex x="42.672" y="9.652"/>
+<vertex x="41.656" y="11.43"/>
+</polygon>
+<wire x1="45.152" y1="12.573" x2="39.624" y2="12.573" width="0.254" layer="1"/>
+<wire x1="39.624" y1="12.573" x2="39.624" y2="12.954" width="0.254" layer="1"/>
 </signal>
 <signal name="ROTBTN">
