File: doc/schematics/licht.sch (EAGLE design)
At the start: 25 parts, among them Q1 MOSFET-NCHANNELFQP30N06L, Q2 MOSFET-PCHANNELSMD

Commit message: toller state
Parts:
- D1: value (none) -> SMD ZD 16; device diode:ZENER-DIODESOT223 -> diode:ZENER-DIODESOT23
- Q2: value MOSFET-PCHANNELSMD -> IRFML8244; device SparkFun-DiscreteSemi:MOSFET-PCHANNELSMD -> SparkFun-DiscreteSemi:MOSFET-PCHANNEL
Changed lines of the file:
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@@
 <part name="P+1" library="supply1" deviceset="V+" device=""/>
 <part name="P+2" library="supply1" deviceset="V+" device=""/>
-<part name="Q2" library="SparkFun-DiscreteSemi" deviceset="MOSFET-PCHANNEL" device="SMD"/>
-<part name="D1" library="diode" deviceset="ZENER-DIODE" device="SOT223"/>
+<part name="Q2" library="SparkFun-DiscreteSemi" deviceset="MOSFET-PCHANNEL" device="" value="IRFML8244"/>
+<part name="D1" library="diode" deviceset="ZENER-DIODE" device="SOT23" value="SMD ZD 16"/>
 <part name="P+3" library="supply1" deviceset="V+" device=""/>
 <part name="R3" library="rcl" deviceset="R-EU_" device="R0805" value="100k"/>

Commit message: Lauter neue Teile
Parts:
- removed D1: SMD ZD 16, diode:ZENER-DIODESOT23
- removed IC1: (no value), SparkFun-PowerIC:V_REG_LM1117SOT223
- removed R3: 100k, rcl:R-EU_R0805
- added IC2: (no value), sprawl:TS2940
- C7: device florolf:CPOL-EUPANASONIC_D-BIGPAD -> florolf:CPOL-EUE2.5-5
- Q2: value IRFML8244 -> IRF7416; device SparkFun-DiscreteSemi:MOSFET-PCHANNEL -> sprawl:IRF7205
Connections:
- removed net N$5: D1.A, Q2.G, R3.2
- net +3V3: now also IC2.OUT; no longer IC1.OUT, IC1.OUT@1
- net GND: now also IC2.GND, Q2.G; no longer IC1.ADJ, R3.1
- net V+: now also IC2.IN; no longer D1.C, IC1.IN
Changed lines of the file:
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@@
 <part name="+3V1" library="supply1" deviceset="+3V3" device=""/>
 <part name="GND1" library="supply1" deviceset="GND" device=""/>
-<part name="IC1" library="SparkFun-PowerIC" deviceset="V_REG_LM1117" device="SOT223"/>
 <part name="+3V2" library="supply1" deviceset="+3V3" device=""/>
 <part name="GND2" library="supply1" deviceset="GND" device=""/>
@@
 <part name="GND4" library="supply1" deviceset="GND" device=""/>
 <part name="L1" library="florolf" deviceset="L-EU" device="PISR-BIGPAD" value="1u"/>
-<part name="C7" library="florolf" deviceset="CPOL-EU" device="PANASONIC_D-BIGPAD" value="100u"/>
+<part name="C7" library="florolf" deviceset="CPOL-EU" device="E2.5-5" value="100u"/>
 <part name="IR1" library="tsop1736" deviceset="TSOP17*TB1" device="" technology="36"/>
 <part name="GND10" library="supply1" deviceset="GND" device=""/>
@@
 <part name="P+1" library="supply1" deviceset="V+" device=""/>
 <part name="P+2" library="supply1" deviceset="V+" device=""/>
-<part name="Q2" library="SparkFun-DiscreteSemi" deviceset="MOSFET-PCHANNEL" device="" value="IRFML8244"/>
-<part name="D1" library="diode" deviceset="ZENER-DIODE" device="SOT23" value="SMD ZD 16"/>
 <part name="P+3" library="supply1" deviceset="V+" device=""/>
-<part name="R3" library="rcl" deviceset="R-EU_" device="R0805" value="100k"/>
 <part name="GND12" library="supply1" deviceset="GND" device=""/>
 <part name="ROTARY" library="con-lstb" deviceset="MA04-1" device=""/>
@@
 <part name="P+4" library="supply1" deviceset="V+" device=""/>
 <part name="F1" library="sprawl" deviceset="PTF45" device=""/>
+<part name="IC2" library="sprawl" deviceset="TS2940" device=""/>
+<part name="Q2" library="sprawl" deviceset="IRF7205" device="" value="IRF7416"/>
 </parts>
 <sheets>
@@
 <instance part="+3V1" gate="G$1" x="25.4" y="119.38"/>
 <instance part="GND1" gate="1" x="7.62" y="96.52"/>
-<instance part="IC1" gate="G$1" x="7.62" y="111.76"/>
 <instance part="+3V2" gate="G$1" x="40.64" y="76.2"/>
 <instance part="GND2" gate="1" x="27.94" y="68.58" rot="R270"/>
@@
 <instance part="P+1" gate="1" x="-10.16" y="119.38"/>
 <instance part="P+2" gate="1" x="152.4" y="124.46"/>
-<instance part="Q2" gate="G$1" x="198.12" y="33.02" rot="R90"/>
-<instance part="D1" gate="G$1" x="208.28" y="25.4" rot="R90"/>
 <instance part="P+3" gate="1" x="220.98" y="33.02" rot="R270"/>
-<instance part="R3" gate="G$1" x="198.12" y="15.24" rot="R90"/>
-<instance part="GND12" gate="1" x="198.12" y="7.62" rot="MR0"/>
+<instance part="GND12" gate="1" x="198.12" y="17.78" rot="MR0"/>
 <instance part="ROTARY" gate="1" x="45.72" y="22.86"/>
 <instance part="GND13" gate="1" x="66.04" y="15.24"/>
@@
 <instance part="P+4" gate="1" x="111.76" y="88.9" rot="R90"/>
 <instance part="F1" gate="1" x="182.88" y="33.02"/>
+<instance part="IC2" gate="1" x="7.62" y="111.76"/>
+<instance part="Q2" gate="G$1" x="195.58" y="27.94" rot="R90"/>
 </instances>
 <busses>
@@
 <net name="GND" class="0">
 <segment>
-<pinref part="IC1" gate="G$1" pin="ADJ"/>
 <pinref part="GND1" gate="1" pin="GND"/>
 <wire x1="7.62" y1="99.06" x2="7.62" y2="101.6" width="0.1524" layer="91"/>
@@
 <wire x1="-10.16" y1="101.6" x2="-5.08" y2="101.6" width="0.1524" layer="91"/>
 <junction x="-5.08" y="101.6"/>
+<pinref part="IC2" gate="1" pin="GND"/>
 </segment>
 <segment>
@@
 </segment>
 <segment>
-<pinref part="R3" gate="G$1" pin="1"/>
-<pinref part="GND12" gate="1" pin="GND"/>
-</segment>
-<segment>
 <pinref part="ROTARY" gate="1" pin="1"/>
 <wire x1="66.04" y1="17.78" x2="53.34" y2="17.78" width="0.1524" layer="91"/>
@@
 <wire x1="17.78" y1="43.18" x2="10.16" y2="43.18" width="0.1524" layer="91"/>
 </segment>
+<segment>
+<wire x1="198.12" y1="22.86" x2="198.12" y2="20.32" width="0.1524" layer="91"/>
+<pinref part="GND12" gate="1" pin="GND"/>
+<pinref part="Q2" gate="G$1" pin="G"/>
+</segment>
 </net>
 <net name="+3V3" class="0">
 <segment>
-<pinref part="IC1" gate="G$1" pin="OUT"/>
 <pinref part="+3V1" gate="G$1" pin="+3V3"/>
 <wire x1="15.24" y1="111.76" x2="17.78" y2="111.76" width="0.1524" layer="91"/>
@@
 <wire x1="20.32" y1="111.76" x2="25.4" y2="111.76" width="0.1524" layer="91"/>
 <wire x1="25.4" y1="111.76" x2="25.4" y2="116.84" width="0.1524" layer="91"/>
-<pinref part="IC1" gate="G$1" pin="OUT@1"/>
 <wire x1="15.24" y1="109.22" x2="17.78" y2="109.22" width="0.1524" layer="91"/>
 <wire x1="17.78" y1="109.22" x2="17.78" y2="111.76" width="0.1524" layer="91"/>
@@
 <pinref part="C1" gate="G$1" pin="1"/>
 <junction x="20.32" y="111.76"/>
+<pinref part="IC2" gate="1" pin="OUT"/>
 </segment>
 <segment>
@@
 <segment>
 <wire x1="193.04" y1="33.02" x2="187.96" y2="33.02" width="0.1524" layer="91"/>
+<pinref part="F1" gate="1" pin="2"/>
 <pinref part="Q2" gate="G$1" pin="D"/>
-<pinref part="F1" gate="1" pin="2"/>
 </segment>
 </net>
 <net name="V+" class="0">
 <segment>
-<pinref part="IC1" gate="G$1" pin="IN"/>
 <wire x1="0" y1="111.76" x2="-5.08" y2="111.76" width="0.1524" layer="91"/>
 <wire x1="-5.08" y1="111.76" x2="-10.16" y2="111.76" width="0.1524" layer="91"/>
@@
 <junction x="-10.16" y="111.76"/>
 <pinref part="P+1" gate="1" pin="V+"/>
+<pinref part="IC2" gate="1" pin="IN"/>
 </segment>
 <segment>
@@
 </segment>
 <segment>
+<wire x1="198.12" y1="33.02" x2="218.44" y2="33.02" width="0.1524" layer="91"/>
+<pinref part="P+3" gate="1" pin="V+"/>
 <pinref part="Q2" gate="G$1" pin="S"/>
-<wire x1="203.2" y1="33.02" x2="208.28" y2="33.02" width="0.1524" layer="91"/>
-<pinref part="D1" gate="G$1" pin="C"/>
-<wire x1="208.28" y1="33.02" x2="218.44" y2="33.02" width="0.1524" layer="91"/>
-<wire x1="208.28" y1="27.94" x2="208.28" y2="33.02" width="0.1524" layer="91"/>
-<junction x="208.28" y="33.02"/>
-<pinref part="P+3" gate="1" pin="V+"/>
 </segment>
 <segment>
@@
 </segment>
 </net>
-<net name="N$5" class="0">
-<segment>
-<pinref part="Q2" gate="G$1" pin="G"/>
-<wire x1="198.12" y1="25.4" x2="198.12" y2="20.32" width="0.1524" layer="91"/>
-<wire x1="198.12" y1="20.32" x2="208.28" y2="20.32" width="0.1524" layer="91"/>
-<pinref part="D1" gate="G$1" pin="A"/>
-<wire x1="208.28" y1="20.32" x2="208.28" y2="22.86" width="0.1524" layer="91"/>
-<pinref part="R3" gate="G$1" pin="2"/>
-<junction x="198.12" y="20.32"/>
-</segment>
-</net>
